File: Schematics/REV3.X/LAMEBOY.sch (EAGLE design)
At the start: 61 parts, among them IC1 PCF8574T, IC3 MCP73831, Q1 12MHz, U1 USD-SOCKETMICROSDEBAY

Commit message: moved 3.1 to 3.X
added pull down power switch
Parts:
- added R14: 10k, rcl:R-EU_ONEFITSALL
Connections:
- net GND: now also R14.2
- net VREG_EN: now also R14.1
Changed lines of the file:
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@@
 <part name="JP1" library="SparkFun-Connectors" deviceset="USB_MICROB_PLUG" device="-IDK"/>
 <part name="GND38" library="supply1" deviceset="GND" device=""/>
+<part name="R14" library="rcl" deviceset="R-EU_" device="ONEFITSALL" value="10k"/>
+<part name="GND39" library="supply1" deviceset="GND" device=""/>
 </parts>
 <sheets>
@@
 <instance part="R7" gate="G$1" x="147.32" y="12.7" rot="R180"/>
 <instance part="GND15" gate="1" x="154.94" y="7.62"/>
+<instance part="R14" gate="G$1" x="149.86" y="48.26" rot="R270"/>
+<instance part="GND39" gate="1" x="149.86" y="38.1"/>
 </instances>
 <busses>
@@
 <pinref part="GND15" gate="1" pin="GND"/>
 <wire x1="154.94" y1="10.16" x2="154.94" y2="12.7" width="0.1524" layer="91"/>
+</segment>
+<segment>
+<pinref part="R14" gate="G$1" pin="2"/>
+<pinref part="GND39" gate="1" pin="GND"/>
+<wire x1="149.86" y1="43.18" x2="149.86" y2="40.64" width="0.1524" layer="91"/>
 </segment>
 </net>
@@
 <wire x1="147.32" y1="60.96" x2="149.86" y2="60.96" width="0.1524" layer="91"/>
 <junction x="149.86" y="60.96"/>
-</segment>
-</net>
+<pinref part="R14" gate="G$1" pin="1"/>
+<wire x1="149.86" y1="55.88" x2="149.86" y2="53.34" width="0.1524" layer="91"/>
+<junction x="149.86" y="55.88"/>
+</segment>
+</net>

Commit message: minor changes to rev3.1
Connections:
- net GPIO0 renamed GPIO0/LCD_RST
- net GPIO15 renamed GPIO15/LCD_CS
- net GPIO2 renamed GPIO2/LCD_DC
Other:
- moved on the sheet: C10, C11, C9
Changed lines of the file:
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@@
 </instance>
 <instance part="U1" gate="G$1" x="172.72" y="121.92"/>
-<instance part="GND28" gate="1" x="157.48" y="104.14" rot="R270"/>
-<instance part="GND29" gate="1" x="157.48" y="106.68" rot="R270"/>
-<instance part="GND30" gate="1" x="157.48" y="111.76" rot="R270"/>
+<instance part="GND28" gate="1" x="160.02" y="104.14" rot="R270"/>
+<instance part="GND29" gate="1" x="160.02" y="106.68" rot="R270"/>
+<instance part="GND30" gate="1" x="160.02" y="111.76" rot="R270"/>
 <instance part="GND31" gate="1" x="157.48" y="121.92" rot="R270"/>
 <instance part="SUPPLY13" gate="G$1" x="157.48" y="127" rot="R90"/>
@@
 <attribute name="NAME" x="53.34" y="71.12" size="1.778" layer="95"/>
 </instance>
-<instance part="C9" gate="G$1" x="144.78" y="68.58" rot="R180"/>
-<instance part="GND12" gate="1" x="144.78" y="60.96"/>
-<instance part="SUPPLY4" gate="G$1" x="144.78" y="76.2"/>
-<instance part="C10" gate="G$1" x="152.4" y="68.58" rot="R180"/>
-<instance part="GND36" gate="1" x="152.4" y="60.96"/>
-<instance part="SUPPLY7" gate="G$1" x="152.4" y="76.2"/>
-<instance part="C11" gate="G$1" x="160.02" y="68.58" rot="R180"/>
-<instance part="GND37" gate="1" x="160.02" y="60.96"/>
-<instance part="SUPPLY11" gate="G$1" x="160.02" y="76.2"/>
+<instance part="C9" gate="G$1" x="144.78" y="55.88" rot="R180"/>
+<instance part="GND12" gate="1" x="144.78" y="48.26"/>
+<instance part="SUPPLY4" gate="G$1" x="144.78" y="63.5"/>
+<instance part="C10" gate="G$1" x="152.4" y="55.88" rot="R180"/>
+<instance part="GND36" gate="1" x="152.4" y="48.26"/>
+<instance part="SUPPLY7" gate="G$1" x="152.4" y="63.5"/>
+<instance part="C11" gate="G$1" x="160.02" y="55.88" rot="R180"/>
+<instance part="GND37" gate="1" x="160.02" y="48.26"/>
+<instance part="SUPPLY11" gate="G$1" x="160.02" y="63.5"/>
 <instance part="JP1" gate="G$1" x="88.9" y="-25.4" smashed="yes" rot="MR0">
 <attribute name="NAME" x="93.726" y="-17.272" size="1.778" layer="95" rot="MR0"/>
@@
 <segment>
 <pinref part="U1" gate="G$1" pin="CD2"/>
-<wire x1="165.1" y1="104.14" x2="160.02" y2="104.14" width="0.1524" layer="91"/>
+<wire x1="165.1" y1="104.14" x2="162.56" y2="104.14" width="0.1524" layer="91"/>
 <pinref part="GND28" gate="1" pin="GND"/>
 </segment>
 <segment>
 <pinref part="U1" gate="G$1" pin="SHIELD@3"/>
-<wire x1="165.1" y1="106.68" x2="160.02" y2="106.68" width="0.1524" layer="91"/>
+<wire x1="165.1" y1="106.68" x2="162.56" y2="106.68" width="0.1524" layer="91"/>
 <pinref part="GND29" gate="1" pin="GND"/>
 </segment>
 <segment>
 <pinref part="U1" gate="G$1" pin="SHIELD@1"/>
-<wire x1="165.1" y1="111.76" x2="160.02" y2="111.76" width="0.1524" layer="91"/>
+<wire x1="165.1" y1="111.76" x2="162.56" y2="111.76" width="0.1524" layer="91"/>
 <pinref part="GND30" gate="1" pin="GND"/>
 </segment>
@@
 <pinref part="C9" gate="G$1" pin="1"/>
 <pinref part="GND12" gate="1" pin="GND"/>
-<wire x1="144.78" y1="66.04" x2="144.78" y2="63.5" width="0.1524" layer="91"/>
+<wire x1="144.78" y1="53.34" x2="144.78" y2="50.8" width="0.1524" layer="91"/>
 </segment>
 <segment>
 <pinref part="C10" gate="G$1" pin="1"/>
 <pinref part="GND36" gate="1" pin="GND"/>
-<wire x1="152.4" y1="66.04" x2="152.4" y2="63.5" width="0.1524" layer="91"/>
+<wire x1="152.4" y1="53.34" x2="152.4" y2="50.8" width="0.1524" layer="91"/>
 </segment>
 <segment>
 <pinref part="C11" gate="G$1" pin="1"/>
 <pinref part="GND37" gate="1" pin="GND"/>
-<wire x1="160.02" y1="66.04" x2="160.02" y2="63.5" width="0.1524" layer="91"/>
+<wire x1="160.02" y1="53.34" x2="160.02" y2="50.8" width="0.1524" layer="91"/>
 </segment>
 <segment>
@@
 <pinref part="C9" gate="G$1" pin="2"/>
 <pinref part="SUPPLY4" gate="G$1" pin="VCC"/>
-<wire x1="144.78" y1="76.2" x2="144.78" y2="73.66" width="0.1524" layer="91"/>
+<wire x1="144.78" y1="63.5" x2="144.78" y2="60.96" width="0.1524" layer="91"/>
 </segment>
 <segment>
 <pinref part="C10" gate="G$1" pin="2"/>
 <pinref part="SUPPLY7" gate="G$1" pin="VCC"/>
-<wire x1="152.4" y1="76.2" x2="152.4" y2="73.66" width="0.1524" layer="91"/>
+<wire x1="152.4" y1="63.5" x2="152.4" y2="60.96" width="0.1524" layer="91"/>
 </segment>
 <segment>
 <pinref part="C11" gate="G$1" pin="2"/>
 <pinref part="SUPPLY11" gate="G$1" pin="VCC"/>
-<wire x1="160.02" y1="76.2" x2="160.02" y2="73.66" width="0.1524" layer="91"/>
+<wire x1="160.02" y1="63.5" x2="160.02" y2="60.96" width="0.1524" layer="91"/>
 </segment>
 </net>
@@
 </segment>
 </net>
-<net name="GPIO15" class="0">
+<net name="GPIO15/LCD_CS" class="0">
 <segment>
 <pinref part="X1" gate="G$1" pin="GPIO15"/>
@@
 </segment>
 </net>
-<net name="GPIO0" class="0">
+<net name="GPIO0/LCD_RST" class="0">
 <segment>
 <pinref part="U$3" gate="G$2" pin="C"/>
@@
 </segment>
 </net>
-<net name="GPIO2" class="0">
+<net name="GPIO2/LCD_DC" class="0">
 <segment>
 <pinref part="RPU" gate="D" pin="2"/>
@@
 <segment>
 <pinref part="U1" gate="G$1" pin="CD1"/>
-<wire x1="165.1" y1="109.22" x2="152.4" y2="109.22" width="0.1524" layer="91"/>
-<label x="152.4" y="109.22" size="1.27" layer="95" rot="R180" xref="yes"/>
-</segment>
-<segment>
+<wire x1="165.1" y1="109.22" x2="157.48" y2="109.22" width="0.1524" layer="91"/>
+<label x="157.48" y="109.22" size="1.27" layer="95" rot="R180" xref="yes"/>
+</segment>
+<segment>
