File: Schematics/REV3.X_CURRENT/LAMEBOY.sch (EAGLE design)
At the start: 62 parts, among them IC1 PCF8574T, IC3 MCP73831, Q1 12MHz, U1 USD-SOCKETMICROSDEBAY

Commit message: minor footprint changes
Changed lines of the file:
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@@
 <wire x1="15.24" y1="71.12" x2="15.24" y2="63.5" width="0.1524" layer="91"/>
 <junction x="15.24" y="71.12"/>
+<junction x="15.24" y="86.36"/>
 </segment>
 <segment>
