File: Schematics/REV2_all_0603/LAMEBOY.brd (EAGLE design)
At the start: 45.7 x 67.3 mm, 60 parts, among them IC1 PCF8574T, IC3 MCP73831, Q1 12MHz, U1 USD-SOCKETMICROSDEBAY, U2 USB

Commit message: moved labels
Routing:
- net VCC: track 254.7 -> 252.8 mm
Changed lines of the file:
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@@
 <contactref element="S2" pad="1"/>
 <wire x1="40.005" y1="52.07" x2="40.767" y2="51.308" width="0.4064" layer="1"/>
-<wire x1="40.767" y1="51.308" x2="40.767" y2="31.75" width="0.4064" layer="1"/>
-<wire x1="26.86091875" y1="31.2592" x2="40.2762" y2="31.2592" width="0.4064" layer="16"/>
-<wire x1="40.2762" y1="31.2592" x2="40.767" y2="31.75" width="0.4064" layer="16"/>
-<via x="40.767" y="31.75" extent="1-16" drill="0.3302" diameter="1.016"/>
+<wire x1="40.767" y1="51.308" x2="40.767" y2="34.29" width="0.4064" layer="1"/>
+<wire x1="26.86091875" y1="31.2592" x2="37.7362" y2="31.2592" width="0.4064" layer="16"/>
+<wire x1="37.7362" y1="31.2592" x2="40.767" y2="34.29" width="0.4064" layer="16"/>
+<via x="40.767" y="34.29" extent="1-16" drill="0.3302" diameter="1.016"/>
 <wire x1="21.86091875" y1="31.2592" x2="21.86091875" y2="34.01908125" width="0.4064" layer="16"/>
 <wire x1="21.86091875" y1="34.01908125" x2="21.59" y2="34.417" width="0.4064" layer="16"/>
@@
 <wire x1="8.121" y1="44.697" x2="8.128" y2="38.735" width="0.4064" layer="1"/>
 <via x="8.128" y="38.735" extent="1-16" drill="0.3302"/>
-<wire x1="40.64" y1="31.877" x2="40.767" y2="31.75" width="0.4064" layer="1"/>
 <wire x1="26.67" y1="32.244" x2="26.67" y2="34.417" width="0.4064" layer="1"/>
 <wire x1="19.685" y1="30.265" x2="21.59" y2="30.265" width="0.4064" layer="1"/>
@@
 <wire x1="34.326" y1="62.194" x2="38.1" y2="58.42" width="0.254" layer="1"/>
 <wire x1="38.1" y1="58.42" x2="38.1" y2="52.07" width="0.254" layer="1"/>
-<wire x1="40.64" y1="31.623" x2="40.767" y2="31.75" width="0.4064" layer="1"/>
 <wire x1="32.315" y1="4.76" x2="34.215" y2="4.76" width="0.4064" layer="1"/>
 <wire x1="34.215" y1="4.76" x2="34.29" y2="4.685" width="0.4064" layer="1"/>
